Commit message: Improved gabeo view

File: panther_gazebo/urdf/description.gazebo.xacro (robot description, xacro)
@@ -29,5 +29,5 @@
   <xacro:arg name="name_space" default="/" />
   <xacro:include filename="$(find panther_description)/urdf/panther.urdf.xacro" />
-  <xacro:include filename="$(find panther_gazebo)/urdf/panther_color.gazebo.xacro" />
+  <xacro:include filename="$(find panther_gazebo)/urdf/materials.gazebo.xacro" />
   <!-- Gazebo plugin for ROS Control -->
   <gazebo>
@@ -38,4 +38,4 @@
   </gazebo>
   <xacro:panther_robot />
-  <xacro:pantker_color_gazebo />
+  <xacro:materials_gazebo />
 </robot>

File: panther_gazebo/urdf/materials.gazebo.xacro (robot description, xacro)
@@ -27,5 +27,5 @@
 <robot name="pantker_color_gazebo" xmlns:xacro="http://ros.org/wiki/xacro">
   <!--<xacro:include filename="$(find panther_gazebo)/urdf/accessories/imu.gazebo.xacro"/>-->
-  <xacro:macro name="pantker_color_gazebo">
+  <xacro:macro name="materials_gazebo">
   <!-- COLOR REFERENCE:
    https://bitbucket.org/osrf/gazebo/src/default/media/materials/scripts/gazebo.material?fileviewer=file-view-default
@@ -47,35 +47,4 @@
     <material>Gazebo/Gold</material>
   </gazebo>
-  <!-- track -->
-  <gazebo reference="track_left_Link">
-    <material>Gazebo/White</material>
-  </gazebo>
-  <gazebo reference="fender_left_Link">
-    <material>Gazebo/Black</material>
-  </gazebo>
-  <gazebo reference="chain_left_Link">
-    <material>Gazebo/Grey</material>
-  </gazebo>
-  <gazebo reference="rubber_left_Link">
-    <material>Gazebo/Black</material>
-  </gazebo>
-  <gazebo reference="sprocket_left_Link">
-    <material>Gazebo/Black</material>
-  </gazebo>
-  <gazebo reference="track_right_Link">
-    <material>Gazebo/White</material>
-  </gazebo>
-  <gazebo reference="fender_right_Link">
-    <material>Gazebo/Black</material>
-  </gazebo>
-  <gazebo reference="chain_right_Link">
-    <material>Gazebo/Grey</material>
-  </gazebo>
-  <gazebo reference="rubber_right_Link">
-    <material>Gazebo/Black</material>
-  </gazebo>
-  <gazebo reference="sprocket_right_Link">
-    <material>Gazebo/Black</material>
-  </gazebo>
   </xacro:macro>
 </robot>

Commit message: First integration zed in simulation

File: panther_gazebo/urdf/description.gazebo.xacro (robot description, xacro)
@@ -30,5 +30,6 @@
   <xacro:include filename="$(find panther_description)/urdf/panther.urdf.xacro" />
   <xacro:include filename="$(find panther_gazebo)/urdf/materials.gazebo.xacro" />
-  <!-- lidar -->
+  <!-- sensors -->
+  <xacro:include filename="$(find panther_gazebo)/urdf/zed.gazebo.xacro" />
   <xacro:include filename="$(find panther_gazebo)/urdf/lidar.gazebo.xacro" />
   <!-- Gazebo plugin for ROS Control -->
@@ -42,3 +43,4 @@
   <xacro:materials_gazebo />
   <xacro:lidar_gazebo />
+  <xacro:zed_camera_gazebo prefix="zed_camera" />
 </robot>

File: panther_gazebo/urdf/zed.gazebo.xacro (robot description, xacro)
@@ -26,41 +26,47 @@
 -->
 <robot xmlns:xacro="http://ros.org/wiki/xacro">
-  <xacro:macro name="lidar_gazebo">
-  <!-- lidar -->
-  <gazebo reference="laser_frame">
-    <sensor type="ray" name="head_hokuyo_sensor">
-      <pose>0 0 0 0 0 0</pose>
-      <visualize>false</visualize>
-      <update_rate>10</update_rate>
-      <ray>
-        <scan>
-          <horizontal>
-            <samples>400</samples>
-            <resolution>1</resolution>
-            <min_angle>-3.14159</min_angle>
-            <max_angle>3.14159</max_angle>
-          </horizontal>
-        </scan>
-        <range>
-          <min>0.10</min>
-          <max>16.0</max>
-          <resolution>0.01</resolution>
-        </range>
-        <noise>
-          <type>gaussian</type>
-          <!-- Noise parameters based on published spec for Hokuyo laser
-               achieving "+-30mm" accuracy at range < 10m.  A mean of 0.0m and
-               stddev of 0.01m will put 99.7% of samples within 0.03m of the true
-               reading. -->
-          <mean>0.0</mean>
-          <stddev>0.01</stddev>
-        </noise>
-      </ray>
-      <plugin name="gazebo_ros_head_hokuyo_controller" filename="libgazebo_ros_laser.so">
-        <topicName>/scan</topicName>
-        <frameName>laser_frame</frameName>
+<xacro:macro name="zed_camera_gazebo" params="prefix">
+  <!--<joint name="${prefix}_joint_optical" type="fixed">
+    <origin xyz="0 0 0" rpy="-1.5708 0 -1.5708"/>
+    <parent link="${prefix}_Link"/>
+    <child link="${prefix}_optical_frame"/>
+  </joint>
+  <link name="${prefix}_optical_frame"/>-->
+  <gazebo reference="zed_depth_frame">
+    <sensor type="depth" name="zed_camera">
+      <always_on>true</always_on>
+      <update_rate>20.0</update_rate>
+      <camera>
+        <horizontal_fov>${58.0*M_PI/180.0}</horizontal_fov>
+        <image>
+          <format>R8G8B8</format>
+          <width>1024</width>
+          <height>768</height>
+        </image>
+        <clip>
+          <near>0.08</near>
+          <far>3.0</far>
+        </clip>
+      </camera>
+      <plugin name="zed_camera_controller" filename="libgazebo_ros_openni_kinect.so">
+        <cameraName>zed_camera</cameraName>
+        <alwaysOn>true</alwaysOn>
+        <updateRate>30</updateRate>
+        <imageTopicName>rgb/image_raw</imageTopicName>
+        <depthImageTopicName>depth/image_raw</depthImageTopicName>
+        <pointCloudTopicName>depth/points</pointCloudTopicName>
+        <cameraInfoTopicName>rgb/camera_info</cameraInfoTopicName>
+        <depthImageCameraInfoTopicName>depth/camera_info</depthImageCameraInfoTopicName>
+        <frameName>zed_depth_frame</frameName>
+        <baseline>0.1</baseline>
+        <distortion_k1>0.0</distortion_k1>
+        <distortion_k2>0.0</distortion_k2>
+        <distortion_k3>0.0</distortion_k3>
+        <distortion_t1>0.0</distortion_t1>
+        <distortion_t2>0.0</distortion_t2>
+        <pointCloudCutoff>0.4</pointCloudCutoff>
       </plugin>
     </sensor>
   </gazebo>
-  </xacro:macro>
+</xacro:macro>
 </robot>

Commit message: Fixed ZED camera emulation

File: panther_gazebo/urdf/description.gazebo.xacro (robot description, xacro)
@@ -43,4 +43,4 @@
   <xacro:materials_gazebo />
   <xacro:lidar_gazebo />
-  <xacro:zed_camera_gazebo prefix="zed_camera" />
+  <xacro:zed_camera_gazebo prefix="zed" />
 </robot>

File: panther_gazebo/urdf/zed.gazebo.xacro (robot description, xacro)
@@ -27,12 +27,61 @@
 <robot xmlns:xacro="http://ros.org/wiki/xacro">
 <xacro:macro name="zed_camera_gazebo" params="prefix">
-  <!--<joint name="${prefix}_joint_optical" type="fixed">
-    <origin xyz="0 0 0" rpy="-1.5708 0 -1.5708"/>
-    <parent link="${prefix}_Link"/>
-    <child link="${prefix}_optical_frame"/>
-  </joint>
-  <link name="${prefix}_optical_frame"/>-->
-  <gazebo reference="zed_depth_frame">
-    <sensor type="depth" name="zed_camera">
+  <gazebo reference="${prefix}_initial_frame">
+    <sensor type="multicamera" name="${prefix}_stereo_camera">
+      <update_rate>30.0</update_rate>
+      <camera name="left">
+        <horizontal_fov>${58.0*M_PI/180.0}</horizontal_fov>
+        <image>
+          <width>3840</width>
+          <height>1080</height>
+          <format>R8G8B8</format>
+        </image>
+        <clip>
+          <near>0.02</near>
+          <far>300</far>
+        </clip>
+        <noise>
+          <type>gaussian</type>
+          <mean>0.0</mean>
+          <stddev>0.007</stddev>
+        </noise>
+      </camera>
+      <camera name="right">
+        <!--<pose>0 -0.07 0 0 0 0</pose>-->
+        <horizontal_fov>${58.0*M_PI/180.0}</horizontal_fov>
+        <image>
+          <width>3840</width>
+          <height>1080</height>
+          <format>R8G8B8</format>
+        </image>
+        <clip>
+          <near>0.02</near>
+          <far>300</far>
+        </clip>
+        <noise>
+          <type>gaussian</type>
+          <mean>0.0</mean>
+          <stddev>0.007</stddev>
+        </noise>
+      </camera>
+      <plugin name="stereo_camera_controller" filename="libgazebo_ros_multicamera.so">
+        <cameraName>${prefix}</cameraName>
+        <alwaysOn>true</alwaysOn>
+        <updateRate>30.0</updateRate>
+        <imageTopicName>image_raw_color</imageTopicName>
+        <cameraInfoTopicName>camera_info</cameraInfoTopicName>
+        <frameName>ZED_left_camera</frameName>
+        <rightFrameName>ZED_right_camera</rightFrameName>
+        <hackBaseline>0.07</hackBaseline>
+        <distortionK1>0.0</distortionK1>
+        <distortionK2>0.0</distortionK2>
+        <distortionK3>0.0</distortionK3>
+        <distortionT1>0.0</distortionT1>
+        <distortionT2>0.0</distortionT2>
+      </plugin>
+    </sensor>
+  </gazebo>
+  <gazebo reference="${prefix}_initial_frame">
+    <sensor type="depth" name="${prefix}_depth">
       <always_on>true</always_on>
       <update_rate>20.0</update_rate>
@@ -41,22 +90,22 @@
         <image>
           <format>R8G8B8</format>
-          <width>1024</width>
-          <height>768</height>
+          <width>3840</width>
+          <height>1080</height>
         </image>
         <clip>
-          <near>0.08</near>
-          <far>3.0</far>
+          <near>0.5</near>
+          <far>20.0</far>
         </clip>
       </camera>
-      <plugin name="zed_camera_controller" filename="libgazebo_ros_openni_kinect.so">
-        <cameraName>zed_camera</cameraName>
+      <plugin name="${prefix}_camera_controller" filename="libgazebo_ros_openni_kinect.so">
+        <cameraName>${prefix}</cameraName>
         <alwaysOn>true</alwaysOn>
         <updateRate>30</updateRate>
-        <imageTopicName>rgb/image_raw</imageTopicName>
-        <depthImageTopicName>depth/image_raw</depthImageTopicName>
+        <imageTopicName>rgb/image_raw_color</imageTopicName>
+        <depthImageTopicName>depth/depth_registered</depthImageTopicName>
         <pointCloudTopicName>depth/points</pointCloudTopicName>
         <cameraInfoTopicName>rgb/camera_info</cameraInfoTopicName>
         <depthImageCameraInfoTopicName>depth/camera_info</depthImageCameraInfoTopicName>
-        <frameName>zed_depth_frame</frameName>
+        <frameName>${prefix}_depth_frame</frameName>
         <baseline>0.1</baseline>
         <distortion_k1>0.0</distortion_k1>
