Commit message: Fix #3 and fix rosinstall

File: panther_gazebo/urdf/imu.gazebo.xacro (robot description, xacro)
@@ -21,5 +21,8 @@
 <robot xmlns:xacro="http://ros.org/wiki/xacro">
   <xacro:macro name="imu_gazebo" params="name frame">
-    <!-- lidar -->
+    <gazebo reference="imu_board_link">
+      <material>Gazebo/Red</material>
+    </gazebo>
+    <!-- IMU -->
     <gazebo reference="base_imu_link">
         <gravity>true</gravity>

File: panther_gazebo/urdf/materials.gazebo.xacro (robot description, xacro)
@@ -23,9 +23,16 @@
     <!-- COLOR REFERENCE:
     https://bitbucket.org/osrf/gazebo/src/default/media/materials/scripts/gazebo.material?fileviewer=file-view-default
+    http://wiki.ros.org/simulator_gazebo/Tutorials/ListOfMaterials
     -->
+    <!--<material>
+      <script>
+        <name>Gazebo/BlueTransparent</name>
+        <uri>file://media/materials/scripts/gazebo.material</uri>
+      </script>
+    </material>-->
     <!-- chassis -->
-    <gazebo reference="cover_link">
-      <material>Gazebo/WhiteGlow</material>
-    </gazebo>
+   <gazebo reference="cover_link">
+     <material>Gazebo/GreyTransparent</material>
+   </gazebo>
     <gazebo reference="iron_link">
       <material>Gazebo/Grey</material>
@@ -40,4 +47,10 @@
       <material>Gazebo/Gold</material>
     </gazebo>
+    <gazebo reference="connectors_link">
+      <material>Gazebo/Black</material>
+    </gazebo>
+    <gazebo reference="battery_link">
+      <material>Gazebo/SkyBlue</material>
+    </gazebo>
     <gazebo reference="stand_link">
       <material>Gazebo/Black</material>

File: panther_gazebo/urdf/zed.gazebo.xacro (robot description, xacro)
@@ -70,4 +70,8 @@
         <xacro:property name="clip_near" value="0.3" />
         <xacro:property name="clip_far" value="25" />
+        <!-- Gazebo color -->
+        <gazebo reference="${camera_model}_camera_center">
+          <material>Gazebo/Grey</material>
+        </gazebo>
     </xacro:if>
     <xacro:if value="${camera_model == 'zedm'}">
@@ -78,4 +82,8 @@
         <!-- Add IMU for ZED -->
         <xacro:imu_gazebo name="${camera_name}" frame="${camera_name}_imu_frame_gazebo" />
+        <!-- Gazebo color -->
+        <gazebo reference="${camera_model}_camera_center">
+          <material>Gazebo/DarkGrey</material>
+        </gazebo>
     </xacro:if>
     <xacro:if value="${camera_model == 'zed2'}">
@@ -86,4 +94,8 @@
         <!-- Add IMU for ZED -->
         <xacro:imu_gazebo name="${camera_name}" frame="${camera_name}_imu_frame_gazebo" />
+        <!-- Gazebo color -->
+        <gazebo reference="${camera_model}_camera_center">
+          <material>Gazebo/Black</material>
+        </gazebo>
     </xacro:if>
     <gazebo reference="${camera_model}_camera_center">
