Commit message: refactoring and License update

File: urdf/description.gazebo.xacro (robot description, xacro)
@@ -1,2 +1,4 @@
+<?xml version="1.0"?>
+<!--
 The MIT License (MIT)
 Copyright (c) 2020 Raffaello Bonghi
@@ -16,2 +18,23 @@
 OUT OF OR IN CONNECTION WITH THE SOFTWARE OR THE USE OR OTHER DEALINGS IN THE
 SOFTWARE.
+-->
+<robot name="panther_robot_gazebo" xmlns:xacro="http://ros.org/wiki/xacro">
+  <!--<xacro:arg name="imu_enabled" default="false" />-->
+  <xacro:arg name="name_space" default="/" />
+  <xacro:include filename="$(find panther_description)/urdf/panther.urdf.xacro" />
+  <xacro:include filename="$(find panther_gazebo)/urdf/materials.gazebo.xacro" />
+  <!-- sensors -->
+  <xacro:include filename="$(find panther_gazebo)/urdf/zed.gazebo.xacro" />
+  <xacro:include filename="$(find panther_gazebo)/urdf/lidar.gazebo.xacro" />
+  <!-- Gazebo plugin for ROS Control -->
+  <gazebo>
+    <plugin name="gazebo_ros_control" filename="libgazebo_ros_control.so">
+      <robotNamespace>/</robotNamespace>
+      <robotSimType>gazebo_ros_control/DefaultRobotHWSim</robotSimType>
+    </plugin>
+  </gazebo>
+  <xacro:panther_robot />
+  <xacro:materials_gazebo />
+  <xacro:lidar_gazebo />
+  <xacro:zed_camera_gazebo prefix="zed" />
+</robot>

File: urdf/materials.gazebo.xacro (robot description, xacro)
@@ -1,2 +1,4 @@
+<?xml version="1.0"?>
+<!--
 The MIT License (MIT)
 Copyright (c) 2020 Raffaello Bonghi
@@ -16,2 +18,33 @@
 OUT OF OR IN CONNECTION WITH THE SOFTWARE OR THE USE OR OTHER DEALINGS IN THE
 SOFTWARE.
+-->
+<robot name="pantker_color_gazebo" xmlns:xacro="http://ros.org/wiki/xacro">
+  <!--<xacro:include filename="$(find panther_gazebo)/urdf/accessories/imu.gazebo.xacro"/>-->
+  <xacro:macro name="materials_gazebo">
+  <!-- COLOR REFERENCE:
+   https://bitbucket.org/osrf/gazebo/src/default/media/materials/scripts/gazebo.material?fileviewer=file-view-default
+  -->
+  <!-- chassis -->
+  <gazebo reference="cover_link">
+    <material>Gazebo/WhiteGlow</material>
+  </gazebo>
+  <gazebo reference="iron_link">
+    <material>Gazebo/Grey</material>
+  </gazebo>
+  <gazebo reference="frame_link">
+    <material>Gazebo/Black</material>
+  </gazebo>
+  <gazebo reference="antenna_link">
+    <material>Gazebo/Black</material>
+  </gazebo>
+  <gazebo reference="speaker_link">
+    <material>Gazebo/Gold</material>
+  </gazebo>
+  <gazebo reference="stand_link">
+    <material>Gazebo/Black</material>
+  </gazebo>
+  <gazebo reference="laser_link">
+    <material>Gazebo/DarkGrey</material>
+  </gazebo>
+  </xacro:macro>
+</robot>

File: urdf/zed.gazebo.xacro (robot description, xacro)
@@ -1,27 +1,21 @@
 <?xml version="1.0"?>
 <!--
-Copyright (C) 2017, Raffaello Bonghi <raffaello@rnext.it>
-All rights reserved
-Redistribution and use in source and binary forms, with or without
-modification, are permitted provided that the following conditions are met:
-1. Redistributions of source code must retain the above copyright
-   notice, this list of conditions and the following disclaimer.
-2. Redistributions in binary form must reproduce the above copyright
-   notice, this list of conditions and the following disclaimer in the
-   documentation and/or other materials provided with the distribution.
-3. Neither the name of the copyright holder nor the names of its
-   contributors may be used to endorse or promote products derived
-   from this software without specific prior written permission.
-THIS SOFTWARE IS PROVIDED BY THE COPYRIGHT HOLDERS AND
-CONTRIBUTORS "AS IS" AND ANY EXPRESS OR IMPLIED WARRANTIES, INCLUDING,
-BUT NOT LIMITED TO, THE IMPLIED WARRANTIES OF MERCHANTABILITY AND FITNESS
-FOR A PARTICULAR PURPOSE ARE DISCLAIMED. IN NO EVENT SHALL THE COPYRIGHT
-HOLDER OR CONTRIBUTORS BE LIABLE FOR ANY DIRECT, INDIRECT, INCIDENTAL,
-SPECIAL, EXEMPLARY, OR CONSEQUENTIAL DAMAGES (INCLUDING, BUT NOT LIMITED TO,
-PROCUREMENT OF SUBSTITUTE GOODS OR SERVICES; LOSS OF USE, DATA, OR PROFITS;
-OR BUSINESS INTERRUPTION) HOWEVER CAUSED AND ON ANY THEORY OF LIABILITY,
-WHETHER IN CONTRACT, STRICT LIABILITY, OR TORT (INCLUDING NEGLIGENCE
-OR OTHERWISE) ARISING IN ANY WAY OUT OF THE USE OF THIS SOFTWARE,
-EVEN IF ADVISED OF THE POSSIBILITY OF SUCH DAMAGE.
+The MIT License (MIT)
+Copyright (c) 2020 Raffaello Bonghi
+Permission is hereby granted, free of charge, to any person obtaining a copy
+of this software and associated documentation files (the "Software"), to deal
+in the Software without restriction, including without limitation the rights
+to use, copy, modify, merge, publish, distribute, sublicense, and/or sell
+copies of the Software, and to permit persons to whom the Software is
+furnished to do so, subject to the following conditions:
+The above copyright notice and this permission notice shall be included in all
+copies or substantial portions of the Software.
+THE SOFTWARE IS PROVIDED "AS IS", WITHOUT WARRANTY OF ANY KIND, EXPRESS OR
+IMPLIED, INCLUDING BUT NOT LIMITED TO THE WARRANTIES OF MERCHANTABILITY,
+FITNESS FOR A PARTICULAR PURPOSE AND NONINFRINGEMENT. IN NO EVENT SHALL THE
+AUTHORS OR COPYRIGHT HOLDERS BE LIABLE FOR ANY CLAIM, DAMAGES OR OTHER
+LIABILITY, WHETHER IN AN ACTION OF CONTRACT, TORT OR OTHERWISE, ARISING FROM,
+OUT OF OR IN CONNECTION WITH THE SOFTWARE OR THE USE OR OTHER DEALINGS IN THE
+SOFTWARE.
 -->
 <robot xmlns:xacro="http://ros.org/wiki/xacro">
