Commit message: Improvements simulation package

File: urdf/lidar.gazebo.xacro (robot description, xacro)
@@ -52,6 +52,6 @@
       </ray>
       <plugin name="gazebo_ros_head_hokuyo_controller" filename="libgazebo_ros_laser.so">
-        <topicName>/scan</topicName>
-        <frameName>laser_frame</frameName>
+        <topicName>scan</topicName>
+        <frameName>/laser_frame</frameName>
       </plugin>
     </sensor>

File: urdf/materials.gazebo.xacro (robot description, xacro)
@@ -20,31 +20,30 @@
 -->
 <robot name="pantker_color_gazebo" xmlns:xacro="http://ros.org/wiki/xacro">
-  <!--<xacro:include filename="$(find panther_gazebo)/urdf/accessories/imu.gazebo.xacro"/>-->
   <xacro:macro name="materials_gazebo">
-  <!-- COLOR REFERENCE:
-   https://bitbucket.org/osrf/gazebo/src/default/media/materials/scripts/gazebo.material?fileviewer=file-view-default
-  -->
-  <!-- chassis -->
-  <gazebo reference="cover_link">
-    <material>Gazebo/WhiteGlow</material>
-  </gazebo>
-  <gazebo reference="iron_link">
-    <material>Gazebo/Grey</material>
-  </gazebo>
-  <gazebo reference="frame_link">
-    <material>Gazebo/Black</material>
-  </gazebo>
-  <gazebo reference="antenna_link">
-    <material>Gazebo/Black</material>
-  </gazebo>
-  <gazebo reference="speaker_link">
-    <material>Gazebo/Gold</material>
-  </gazebo>
-  <gazebo reference="stand_link">
-    <material>Gazebo/Black</material>
-  </gazebo>
-  <gazebo reference="laser_link">
-    <material>Gazebo/DarkGrey</material>
-  </gazebo>
+    <!-- COLOR REFERENCE:
+    https://bitbucket.org/osrf/gazebo/src/default/media/materials/scripts/gazebo.material?fileviewer=file-view-default
+    -->
+    <!-- chassis -->
+    <gazebo reference="cover_link">
+      <material>Gazebo/WhiteGlow</material>
+    </gazebo>
+    <gazebo reference="iron_link">
+      <material>Gazebo/Grey</material>
+    </gazebo>
+    <gazebo reference="frame_link">
+      <material>Gazebo/Black</material>
+    </gazebo>
+    <gazebo reference="antenna_link">
+      <material>Gazebo/Black</material>
+    </gazebo>
+    <gazebo reference="speaker_link">
+      <material>Gazebo/Gold</material>
+    </gazebo>
+    <gazebo reference="stand_link">
+      <material>Gazebo/Black</material>
+    </gazebo>
+    <gazebo reference="laser_link">
+      <material>Gazebo/DarkGrey</material>
+    </gazebo>
   </xacro:macro>
 </robot>

File: urdf/panther.gazebo.xacro (robot description, xacro)
@@ -19,22 +19,35 @@
 SOFTWARE.
 -->
-<robot name="panther_robot_gazebo" xmlns:xacro="http://ros.org/wiki/xacro">
+<robot name="sim_panther" xmlns:xacro="http://ros.org/wiki/xacro">
   <!--<xacro:arg name="imu_enabled" default="false" />-->
-  <xacro:arg name="name_space" default="/" />
-  <xacro:include filename="$(find panther_description)/urdf/panther.urdf.xacro" />
-  <xacro:include filename="$(find panther_gazebo)/urdf/materials.gazebo.xacro" />
+  <xacro:arg name="name_space" default="/panther" />
+  <!-- Arguments -->
+  <xacro:arg name="zed_model"   default="zed2"/> <!-- Follow zed_repository -->
+  <xacro:arg name="jetson"      default="xavier"/> <!-- options: tx, xavier -->
+  <xacro:arg name="motor_board" default="roboteq"/> <!-- options: unav, roboteq -->
+  <xacro:arg name="ssd"         default="false"/>
+  <xacro:include filename="$(find panther_description)/urdf/robot.urdf.xacro" />
+  <xacro:include filename="$(find panther_simulation)/urdf/materials.gazebo.xacro" />
   <!-- sensors -->
-  <xacro:include filename="$(find panther_gazebo)/urdf/zed.gazebo.xacro" />
-  <xacro:include filename="$(find panther_gazebo)/urdf/lidar.gazebo.xacro" />
+  <xacro:include filename="$(find panther_simulation)/urdf/zed.gazebo.xacro" />
+  <xacro:include filename="$(find panther_simulation)/urdf/lidar.gazebo.xacro" />
   <!-- Gazebo plugin for ROS Control -->
   <gazebo>
     <plugin name="gazebo_ros_control" filename="libgazebo_ros_control.so">
-      <robotNamespace>/</robotNamespace>
+      <robotNamespace>$(arg name_space)</robotNamespace>
       <robotSimType>gazebo_ros_control/DefaultRobotHWSim</robotSimType>
     </plugin>
   </gazebo>
-  <xacro:panther_robot />
+  <!-- Color materials for Gazebo -->
   <xacro:materials_gazebo />
+  <!-- ZED emulation -->
+  <xacro:zed_camera_gazebo prefix="zed" />
+  <!-- LIDAR emulation -->
   <xacro:lidar_gazebo />
-  <xacro:zed_camera_gazebo prefix="zed" />
+  <!-- Panther robot -->
+  <xacro:panther
+              zed_model="$(arg zed_model)"
+              jetson="$(arg jetson)"
+              motor_board="$(arg motor_board)"
+              ssd="$(arg ssd)" />
 </robot>
