Commit message: Fix ZED simulation #4

File: urdf/panther.gazebo.xacro (robot description, xacro)
@@ -28,4 +28,7 @@
   <xacro:arg name="ssd"         default="false"/>
   <xacro:arg name="ultrasounds"  default="false"/>
+  <xacro:arg name="camera_name"  default="zed"/>
+  <xacro:arg name="depth_camera"  default="left"/>
+  <xacro:arg name="resolution"  default="HD1080"/>
   <xacro:include filename="$(find panther_description)/urdf/robot.urdf.xacro" />
   <xacro:include filename="$(find panther_simulation)/urdf/materials.gazebo.xacro" />
@@ -42,8 +45,4 @@
   <!-- Color materials for Gazebo -->
   <xacro:materials_gazebo />
-  <!-- ZED emulation -->
-  <xacro:zed_camera_gazebo prefix="zed" />
-  <!-- LIDAR emulation -->
-  <xacro:lidar_gazebo />
   <!-- Panther robot -->
   <xacro:panther
@@ -53,3 +52,8 @@
               ssd="$(arg ssd)"
               ultrasounds="$(arg ultrasounds)" />
+  <!-- ZED emulation -->
+  <xacro:zed_camera_gazebo camera_name="$(arg camera_name)" camera_model="$(arg zed_model)"
+                            depth_camera="$(arg depth_camera)" resolution="$(arg resolution)" />
+  <!-- LIDAR emulation -->
+  <xacro:lidar_gazebo />
 </robot>

File: urdf/zed.gazebo.xacro (robot description, xacro)
@@ -1,3 +1,3 @@
-<?xml version="1.0"?>
+<?xml version="1.0" encoding="UTF-8"?>
 <!--
 The MIT License (MIT)
@@ -20,96 +20,149 @@
 -->
 <robot xmlns:xacro="http://ros.org/wiki/xacro">
-<xacro:macro name="zed_camera_gazebo" params="prefix">
-  <gazebo reference="${prefix}_initial_frame">
-    <sensor type="multicamera" name="${prefix}_stereo_camera">
-      <update_rate>30.0</update_rate>
-      <camera name="left">
-        <horizontal_fov>${58.0*M_PI/180.0}</horizontal_fov>
-        <image>
-          <width>3840</width>
-          <height>1080</height>
-          <format>R8G8B8</format>
-        </image>
-        <clip>
-          <near>0.02</near>
-          <far>300</far>
-        </clip>
-        <noise>
-          <type>gaussian</type>
-          <mean>0.0</mean>
-          <stddev>0.007</stddev>
-        </noise>
-      </camera>
-      <camera name="right">
-        <!--<pose>0 -0.07 0 0 0 0</pose>-->
-        <horizontal_fov>${58.0*M_PI/180.0}</horizontal_fov>
-        <image>
-          <width>3840</width>
-          <height>1080</height>
-          <format>R8G8B8</format>
-        </image>
-        <clip>
-          <near>0.02</near>
-          <far>300</far>
-        </clip>
-        <noise>
-          <type>gaussian</type>
-          <mean>0.0</mean>
-          <stddev>0.007</stddev>
-        </noise>
-      </camera>
-      <plugin name="stereo_camera_controller" filename="libgazebo_ros_multicamera.so">
-        <cameraName>${prefix}</cameraName>
-        <alwaysOn>true</alwaysOn>
-        <updateRate>30.0</updateRate>
-        <imageTopicName>image_raw_color</imageTopicName>
-        <cameraInfoTopicName>camera_info</cameraInfoTopicName>
-        <frameName>ZED_left_camera</frameName>
-        <rightFrameName>ZED_right_camera</rightFrameName>
-        <hackBaseline>0.07</hackBaseline>
-        <distortionK1>0.0</distortionK1>
-        <distortionK2>0.0</distortionK2>
-        <distortionK3>0.0</distortionK3>
-        <distortionT1>0.0</distortionT1>
-        <distortionT2>0.0</distortionT2>
-      </plugin>
-    </sensor>
-  </gazebo>
-  <gazebo reference="${prefix}_initial_frame">
-    <sensor type="depth" name="${prefix}_depth">
-      <always_on>true</always_on>
-      <update_rate>20.0</update_rate>
-      <camera>
-        <horizontal_fov>${58.0*M_PI/180.0}</horizontal_fov>
-        <image>
-          <format>R8G8B8</format>
-          <width>3840</width>
-          <height>1080</height>
-        </image>
-        <clip>
-          <near>0.5</near>
-          <far>20.0</far>
-        </clip>
-      </camera>
-      <plugin name="${prefix}_camera_controller" filename="libgazebo_ros_openni_kinect.so">
-        <cameraName>${prefix}</cameraName>
-        <alwaysOn>true</alwaysOn>
-        <updateRate>30</updateRate>
-        <imageTopicName>rgb/image_raw_color</imageTopicName>
-        <depthImageTopicName>depth/depth_registered</depthImageTopicName>
-        <pointCloudTopicName>depth/points</pointCloudTopicName>
-        <cameraInfoTopicName>rgb/camera_info</cameraInfoTopicName>
-        <depthImageCameraInfoTopicName>depth/camera_info</depthImageCameraInfoTopicName>
-        <frameName>${prefix}_depth_frame</frameName>
-        <baseline>0.1</baseline>
-        <distortion_k1>0.0</distortion_k1>
-        <distortion_k2>0.0</distortion_k2>
-        <distortion_k3>0.0</distortion_k3>
-        <distortion_t1>0.0</distortion_t1>
-        <distortion_t2>0.0</distortion_t2>
-        <pointCloudCutoff>0.4</pointCloudCutoff>
-      </plugin>
-    </sensor>
-  </gazebo>
-</xacro:macro>
+  <!-- depth_camera:
+       - left
+       - right
+       -->
+  <xacro:macro name="zed_camera_gazebo" params="camera_name camera_model depth_camera resolution">
+    <xacro:property name="depth_rate" value="100" />
+    <xacro:if value="${resolution == 'HD2K'}">
+        <xacro:property name="resolution_width" value="4416" />
+        <xacro:property name="resolution_heigth" value="1242" />
+        <xacro:property name="update_rate" value="15" />
+    </xacro:if>
+    <xacro:if value="${resolution == 'HD1080'}">
+        <xacro:property name="resolution_width" value="3840" />
+        <xacro:property name="resolution_heigth" value="1080" />
+        <xacro:property name="update_rate" value="30" />
+    </xacro:if>
+    <xacro:if value="${camera_model == 'HD720'}">
+        <xacro:property name="resolution_width" value="2560" />
+        <xacro:property name="resolution_heigth" value="720" />
+        <xacro:property name="update_rate" value="60" />
+    </xacro:if>
+    <xacro:if value="${camera_model == 'VGA'}">
+        <xacro:property name="resolution_width" value="1344" />
+        <xacro:property name="resolution_heigth" value="376" />
+        <xacro:property name="update_rate" value="100" />
+    </xacro:if>
+    <xacro:if value="${camera_model == 'zed'}">
+        <xacro:property name="baseline" value="0.12" />
+        <xacro:property name="fov" value="2.0" />
+        <xacro:property name="clip_near" value="0.3" />
+        <xacro:property name="clip_far" value="25" />
+    </xacro:if>
+    <xacro:if value="${camera_model == 'zedm'}">
+        <xacro:property name="baseline" value="0.06" />
+        <xacro:property name="fov" value="2.0" />
+        <xacro:property name="clip_near" value="0.1" />
+        <xacro:property name="clip_far" value="15" />
+    </xacro:if>
+    <xacro:if value="${camera_model == 'zed2'}">
+        <xacro:property name="baseline" value="0.12" />
+        <xacro:property name="fov" value="1.8" />
+        <xacro:property name="clip_near" value="0.2" />
+        <xacro:property name="clip_far" value="20" />
+    </xacro:if>
+    <link name="camera_depth_frame_gazebo" />
+    <joint name="gazebo_joint" type="fixed">
+      <origin xyz="0 0 0" rpy="${-M_PI/2} 0 ${-M_PI/2}" />
+      <parent link="${camera_model}_${depth_camera}_camera_frame" />
+      <child link="camera_depth_frame_gazebo" />
+    </joint>
+    <gazebo reference="${camera_model}_camera_center">
+      <sensor type="multicamera" name="${camera_name}_stereo_camera">
+        <update_rate>${update_rate}</update_rate>
+        <camera name="left">
+          <horizontal_fov>${58.0*M_PI/180.0}</horizontal_fov>
+          <image>
+            <width>${resolution_width}</width>
+            <height>${resolution_heigth}</height>
+            <format>R8G8B8</format>
+          </image>
+          <clip>
+            <near>0.02</near>
+            <far>300</far>
+          </clip>
+          <noise>
+            <type>gaussian</type>
+            <mean>0.0</mean>
+            <stddev>0.007</stddev>
+          </noise>
+        </camera>
+        <camera name="right">
+          <horizontal_fov>${58.0*M_PI/180.0}</horizontal_fov>
+          <image>
+            <width>${resolution_width}</width>
+            <height>${resolution_heigth}</height>
+            <format>R8G8B8</format>
+          </image>
+          <clip>
+            <near>0.02</near>
+            <far>300</far>
+          </clip>
+          <noise>
+            <type>gaussian</type>
+            <mean>0.0</mean>
+            <stddev>0.007</stddev>
+          </noise>
+        </camera>
+        <plugin name="stereo_camera_controller" filename="libgazebo_ros_multicamera.so">
+          <cameraName>${camera_name}</cameraName>
+          <alwaysOn>true</alwaysOn>
+          <updateRate>${update_rate}</updateRate>
+          <imageTopicName>image_raw_color</imageTopicName>
+          <cameraInfoTopicName>camera_info</cameraInfoTopicName>
+          <frameName>${camera_model}_left_camera_optical_frame</frameName>
+          <rightFrameName>${camera_model}_right_camera_optical_frame</rightFrameName>
+          <hackBaseline>0.07</hackBaseline>
+          <distortionK1>0.0</distortionK1>
+          <distortionK2>0.0</distortionK2>
+          <distortionK3>0.0</distortionK3>
+          <distortionT1>0.0</distortionT1>
+          <distortionT2>0.0</distortionT2>
+        </plugin>
+      </sensor>
+    </gazebo>
+    <gazebo reference="${camera_model}_camera_center">
+      <sensor type="depth" name="${camera_name}_depth">
+        <always_on>true</always_on>
+        <update_rate>${depth_rate}</update_rate>
+        <camera>
+          <horizontal_fov>${fov}</horizontal_fov>
+          <image>
+            <format>R8G8B8</format>
+            <width>${resolution_width}</width>
+            <height>${resolution_heigth}</height>
+          </image>
+          <clip>
+            <near>${clip_near}</near>
+            <far>${clip_far}</far>
+          </clip>
+        </camera>
+        <plugin name="${camera_name}_camera_controller" filename="libgazebo_ros_openni_kinect.so">
+          <cameraName>${camera_name}</cameraName>
+          <alwaysOn>true</alwaysOn>
+          <updateRate>${depth_rate}</updateRate>
+          <imageTopicName>${depth_camera}/image_rect_color</imageTopicName>
+          <depthImageTopicName>depth/depth_registered</depthImageTopicName>
+          <pointCloudTopicName>depth/points</pointCloudTopicName>
+          <cameraInfoTopicName>${depth_camera}/camera_info</cameraInfoTopicName>
+          <depthImageCameraInfoTopicName>depth/camera_info</depthImageCameraInfoTopicName>
+          <frameName>camera_depth_frame_gazebo</frameName>
+          <baseline>${baseline}</baseline>
+          <pointCloudCutoff>0.02</pointCloudCutoff>
+          <distortionK1>0</distortionK1>
+          <distortionK2>0</distortionK2>
+          <distortionK3>0</distortionK3>
+          <distortionT1>0</distortionT1>
+          <distortionT2>0</distortionT2>
+          <CxPrime>0</CxPrime>
+          <Cx>0</Cx>
+          <Cy>0</Cy>
+          <focalLength>0</focalLength>
+          <hackBaseline>0</hackBaseline>
+        </plugin>
+      </sensor>
+    </gazebo>
+  </xacro:macro>
 </robot>

Commit message: Minor fixes emulation ZED

File: urdf/panther.gazebo.xacro (robot description, xacro)
@@ -21,14 +21,24 @@
 <robot name="sim_panther" xmlns:xacro="http://ros.org/wiki/xacro">
   <!--<xacro:arg name="imu_enabled" default="false" />-->
-  <xacro:arg name="name_space" default="/panther" />
+  <xacro:arg name="name_space"  default="/panther" />
   <!-- Arguments -->
-  <xacro:arg name="zed_model"   default="zed2"/> <!-- Follow zed_repository -->
-  <xacro:arg name="jetson"      default="xavier"/> <!-- options: tx, xavier -->
-  <xacro:arg name="motor_board" default="roboteq"/> <!-- options: unav, roboteq -->
-  <xacro:arg name="ssd"         default="false"/>
+  <xacro:arg name="zed_model"    default="zed2"/> <!-- Follow zed_repository -->
+  <xacro:arg name="jetson"       default="xavier"/> <!-- options: tx, xavier -->
+  <xacro:arg name="motor_board"  default="roboteq"/> <!-- options: unav, roboteq -->
+  <xacro:arg name="ssd"          default="false"/>
   <xacro:arg name="ultrasounds"  default="false"/>
-  <xacro:arg name="camera_name"  default="zed"/>
+  <!-- Reference: https://www.stereolabs.com/
+       depth_camera:
+        - left
+        - right
+       resolution:
+        - HD2K
+        - HD1080
+        - HD720
+        - VGA
+       -->
+  <xacro:arg name="camera_name"   default="zed"/>
   <xacro:arg name="depth_camera"  default="left"/>
-  <xacro:arg name="resolution"  default="HD1080"/>
+  <xacro:arg name="resolution"    default="HD720"/>
   <xacro:include filename="$(find panther_description)/urdf/robot.urdf.xacro" />
   <xacro:include filename="$(find panther_simulation)/urdf/materials.gazebo.xacro" />

File: urdf/zed.gazebo.xacro (robot description, xacro)
@@ -20,10 +20,16 @@
 -->
 <robot xmlns:xacro="http://ros.org/wiki/xacro">
-  <!-- depth_camera:
-       - left
-       - right
+  <!-- Reference: https://www.stereolabs.com/
+       depth_camera:
+        - left
+        - right
+       resolution:
+        - HD2K
+        - HD1080
+        - HD720
+        - VGA
        -->
   <xacro:macro name="zed_camera_gazebo" params="camera_name camera_model depth_camera resolution">
-    <xacro:property name="depth_rate" value="100" />
+    <xacro:property name="depth_rate" value="30" />
     <xacro:if value="${resolution == 'HD2K'}">
         <xacro:property name="resolution_width" value="4416" />
@@ -36,10 +42,10 @@
         <xacro:property name="update_rate" value="30" />
     </xacro:if>
-    <xacro:if value="${camera_model == 'HD720'}">
+    <xacro:if value="${resolution == 'HD720'}">
         <xacro:property name="resolution_width" value="2560" />
         <xacro:property name="resolution_heigth" value="720" />
         <xacro:property name="update_rate" value="60" />
     </xacro:if>
-    <xacro:if value="${camera_model == 'VGA'}">
+    <xacro:if value="${resolution == 'VGA'}">
         <xacro:property name="resolution_width" value="1344" />
         <xacro:property name="resolution_heigth" value="376" />
