Commit message: Fix Imu and add on ZED

File: urdf/imu.gazebo.xacro (robot description, xacro)
@@ -20,5 +20,5 @@
 -->
 <robot xmlns:xacro="http://ros.org/wiki/xacro">
-  <xacro:macro name="imu_gazebo" params="name">
+  <xacro:macro name="imu_gazebo" params="name frame">
     <!-- lidar -->
     <gazebo reference="base_imu_link">
@@ -31,10 +31,10 @@
             <plugin filename="libgazebo_ros_imu_sensor.so" name="imu_plugin">
                 <topicName>/${name}/imu/data</topicName>
-                <bodyName>base_imu_link</bodyName>
+                <bodyName>${frame}</bodyName>
                 <updateRateHZ>100.0</updateRateHZ>
                 <gaussianNoise>0.0025</gaussianNoise>
                 <xyzOffset>0 0 0</xyzOffset>
                 <rpyOffset>0 0 0</rpyOffset>
-                <frameName>base_imu_link</frameName>
+                <frameName>${frame}</frameName>
             </plugin>
             <pose>0 0 0 0 0 0</pose>

File: urdf/panther.gazebo.xacro (robot description, xacro)
@@ -68,4 +68,4 @@
   <xacro:lidar_gazebo />
   <!-- IMU emulation -->
-  <xacro:imu_gazebo name="razor" />
+  <xacro:imu_gazebo name="razor" frame="base_imu_link" />
 </robot>

File: urdf/zed.gazebo.xacro (robot description, xacro)
@@ -31,4 +31,17 @@
        -->
   <xacro:macro name="zed_camera_gazebo" params="camera_name camera_model depth_camera resolution">
+    <link name="camera_depth_frame_gazebo" />
+    <joint name="${camera_name}_depth_gazebo_joint" type="fixed">
+      <origin xyz="0 0 0" rpy="${-M_PI/2} 0 ${-M_PI/2}" />
+      <parent link="${camera_model}_${depth_camera}_camera_frame" />
+      <child link="camera_depth_frame_gazebo" />
+    </joint>
+    <!-- TODO: Fix with proper frame -->
+    <link name="${camera_name}_imu_frame_gazebo" />
+    <joint name="${camera_name}_imu_gazebo_joint" type="fixed">
+      <origin xyz="0 0 0" rpy="0 0 0" />
+      <parent link="${camera_model}_camera_center" />
+      <child link="${camera_name}_imu_frame_gazebo" />
+    </joint>
     <xacro:property name="depth_rate" value="30" />
     <xacro:if value="${resolution == 'HD2K'}">
@@ -63,4 +76,6 @@
         <xacro:property name="clip_near" value="0.1" />
         <xacro:property name="clip_far" value="15" />
+        <!-- Add IMU for ZED -->
+        <xacro:imu_gazebo name="${camera_name}" frame="${camera_name}_imu_frame_gazebo" />
     </xacro:if>
     <xacro:if value="${camera_model == 'zed2'}">
@@ -69,11 +84,7 @@
         <xacro:property name="clip_near" value="0.2" />
         <xacro:property name="clip_far" value="20" />
+        <!-- Add IMU for ZED -->
+        <xacro:imu_gazebo name="${camera_name}" frame="${camera_name}_imu_frame_gazebo" />
     </xacro:if>
-    <link name="camera_depth_frame_gazebo" />
-    <joint name="gazebo_joint" type="fixed">
-      <origin xyz="0 0 0" rpy="${-M_PI/2} 0 ${-M_PI/2}" />
-      <parent link="${camera_model}_${depth_camera}_camera_frame" />
-      <child link="camera_depth_frame_gazebo" />
-    </joint>
     <gazebo reference="${camera_model}_camera_center">
       <sensor type="multicamera" name="${camera_name}_stereo_camera">
